File: design/makey_makey.sch (EAGLE design)
At the start: 67 parts, among them U1 ATMEGA32U4TQFP, X1 USBSMD, Y1 16MHz

Commit message: v1.2 of MaKey MaKey renamed files to remove version number
Parts:
- removed J1, J4: (no value), SparkFun-Connectors:M08SMD-COMBO
- removed JP4: (no value), SparkFun-Connectors:M06SMD-STRAIGHT-COMBO
- added JP12, JP13, JP14: (no value), SparkFun-Connectors:M06SMD-STRAIGHT-COMBO
- added LED10, LED11: RED, SparkFun-LED:LED0603
- added LED8, LED9: GREEN, SparkFun-LED:LED0603
- added R18: 330, SparkFun-Passives:RESISTOR0402-RES
- added R19: 1k, SparkFun-Passives:RESISTOR0402-RES
- LED7: value Red -> RED
- R10, R11, R12, R13, R14, R15, R24, R25, R26, R27, R28, R29, R4, R5, R6, R7, R8, R9: value 50M -> 22M
- R16: value 50M -> 1k; device SparkFun:RESISTOR0402-RES -> SparkFun-Passives:RESISTOR0402-RES
- R17: value 50M -> 330; device SparkFun:RESISTOR0402-RES -> SparkFun-Passives:RESISTOR0402-RES
- R23: value 1K -> 1k
- U$1: value OSHW-LOGOL -> OSHW-LOGOM; device SparkFun-Aesthetics:OSHW-LOGOL -> SparkFun-Aesthetics:OSHW-LOGOM
- renumbered A to LEFT, D to RIGHT, S to DOWN, W to UP
Connections:
- new net N$10: LED10.A, R19.1
- new net N$11: LED9.A, R17.1
- new net N$9: LED11.A, R16.1
- new net PD5: LED11.C, LED9.C, U1.PD5
- new net PULL-UP: R10.2, R11.2, R12.2, R13.2, R14.2, R15.2, R4.2, R5.2, R6.2, R7.2, R8.2, R9.2, SJ1.2
- net A0: now also JP12.1; no longer J4.3
- net A1: now also JP12.2; no longer J4.4
- net A2: now also JP12.3; no longer J4.5
- net A3: now also JP12.4; no longer J4.6
- net A4: now also JP12.5; no longer J4.7
- net A5: now also JP12.6; no longer J4.8
- net D0: now also JP13.6; no longer J1.1
- net D1: now also JP13.5; no longer J1.2
- net D12: now also R24.1, UP.1; no longer LEFT.1, R25.1
- net D13: now also LEFT.1, R25.1; no longer DOWN.1, R26.1
- net D14: now also JP14.6; no longer CLICK.1, JP4.3, R29.1
- net D15: now also JP14.1; no longer JP4.4
- net D16: now also JP14.5; no longer JP4.6, R28.1, SPACE.1
- net D17: now also LED10.C, LED8.C; no longer R24.1, UP.1
- net D2: now also JP13.4; no longer J1.3
- net D3: now also JP13.3; no longer J1.4
- net D4: now also JP13.2; no longer J1.5
- net D5: now also JP13.1; no longer J1.6
- net D6: now also CLICK.1, R29.1; no longer J1.7, R16.1
- net D7: now also R28.1, SPACE.1; no longer J1.8, R17.1
- net D8: now also DOWN.1, R26.1
- net GND: now also JP14.3; no longer JP4.1
- net N$3: now also LED8.A, R18.1; no longer R10.2, R11.2, R12.2, R13.2, R14.2, R15.2, R16.2, R17.2, R4.2, R5.2, R6.2, R7.2, R8.2, R9.2, SJ1.2
- net RESET: now also JP14.2; no longer JP4.5
- net VCC: now also JP14.4, R16.2, R17.2, R18.2, R19.2; no longer JP4.2
Other:
- note added: "Jim Lindblom, Jay Silver, Eric Rosenbaum"
- note removed: "Jim Lindblom"
- moved on the sheet: JP3, R16, R17
